File: Clock/Clock.kicad_sch (KiCad schematic)
At the start: 46 parts, among them J1 LED, J2 BUS LEDs, J3 USB_B_Micro, SW1 Pulse, SW2 SW_SPDT, SW3 Reset, U1 TLC555xP, U2 TLC555xP, U3 TLC555xP, U4 74HC14, U5 74LS08, U6 74LS32

Commit message: Initial version of Registers Schematic
Essentially complete and has footprints.
Parts:
- added R17: 2K, Resistor_SMD:R_0805_2012Metric_Pad1.20x1.40mm_HandSolder, symbol Device:R_Small
Connections:
- net GND: now also C6.2, C7.2, SW1.1, R17.1
- net HALT: now also R17.2

Commit message: Updated to v2.0. Sent to manufacturing after review.
Parts:
- removed J3: USB_B_Micro, Connector_USB:USB_Micro-AB_Molex_47590-0001, symbol Connector:USB_B_Micro
- added C14: .33uF, Capacitor_THT:CP_Radial_D5.0mm_P2.50mm, symbol Device:C_Polarized_Small
- added J4: Jack, Connector_BarrelJack:BarrelJack_Horizontal, symbol Connector:Barrel_Jack_MountingPin
- added U7: LM7805_TO220, Package_TO_SOT_THT:TO-220-3_Vertical, symbol Regulator_Linear:LM7805_TO220
- B1, B2, B3: value ~ -> (none)
Connections:
- net GND: now also C14.2, J4.2, U7.2 (GND)
- net 5V renamed +5V
- net +5V: now also U7.3 (VO)
- new net: C14.1, J4.1, U7.1 (VI)
- no-connect marks 11 -> 8
Other:
- moved on the sheet: C10, C9, J1, J2, R10, R11, R12, R13, R14, R15, R17, R8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
