File: Clock/Clock.kicad_sch (KiCad schematic)
At the start: 49 parts, among them J1 LED, J2 BUS LEDs, J4 Jack, SW1 Pulse, SW2 SW_SPDT, SW3 Reset, U1 TLC555xP, U2 TLC555xP, U3 TLC555xP, U4 74HC14, U5 74LS08, U6 74LS32, U7 LM7805_TO220

Commit message: [Clock] - Added horizontal voltage regulator and made more room for tall components.
Parts:
- U7: footprint Package_TO_SOT_THT:TO-220-3_Vertical -> Package_TO_SOT_THT:TO-220F-3_Horizontal_TabDown
Changed lines of the file:
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@@
 			)
 		)
-		(property "Footprint" "Package_TO_SOT_THT:TO-220-3_Vertical"
+		(property "Footprint" "Package_TO_SOT_THT:TO-220F-3_Horizontal_TabDown"
 			(at 264.16 120.015 0)
 			(hide yes)
