File: Clock/Clock.kicad_pcb (KiCad board)
At the start: 2 copper layers, 86.2 x 99.9 mm, 49 parts, among them J1 LED, J2 BUS LEDs, J4 DC Input 12V Max, SW1 Pulse, SW2 SW_SPDT, SW3 Reset, U1 TLC555xP, U2 TLC555xP, U3 TLC555xP, U4 74HC14, U5 74LS08, U6 74LS32, U7 LM7805_TO220

Commit message: [Clock] - Added horizontal voltage regulator and made more room for tall components.
Parts:
- J4: value DC Input 12V Max -> 12V Max Input
- U7: footprint Package_TO_SOT_THT:TO-220-3_Vertical -> Package_TO_SOT_THT:TO-220F-3_Horizontal_TabDown
- moved C12 7.40 mm to (78.5, 106.5)
- moved C11 6.10 mm to (66.5, 103.2), turned to -90 degrees
- moved C14 4.72 mm to (70.8, 121.3), turned to -90 degrees
- moved U7 3.66 mm to (78.3, 116.3)
- moved C5 3.05 mm to (88.5, 57.2), turned to 90 degrees
Routing:
- net GND: track 110.0 -> 104.2 mm
- net Net-(U7-VI): track 21.9 -> 18.7 mm
- net 5V: track 531.1 -> 528.7 mm
- net Net-(U1-THR): track 40.3 -> 38.6 mm
Other:
- board text added: "8-Bit Computer Clock Module v2.1 D. Q. McDonald July 2026"
- board text removed: "5V"
- board text removed: "8-Bit Computer Clock Module v2.0 D. Q. McDonald May 2026"
- board text removed: "COUO"
