File: ALU/ALU.kicad_sch (KiCad schematic)
At the start: 29 parts, among them U1 74HC283, U2 74HC283, U3 74HC245, U4 74HC86, U5 74HC86

Commit message: [ALU] - First fully routed and reviewed version of the ALU.
Parts:
- C1: footprint (none) -> Capacitor_SMD:C_0805_2012Metric_Pad1.18x1.45mm_HandSolder; Autoroute-decouple (none) -> U3
- C2: footprint (none) -> Capacitor_SMD:C_0805_2012Metric_Pad1.18x1.45mm_HandSolder; Autoroute-decouple (none) -> U1
- C3: footprint (none) -> Capacitor_SMD:C_0805_2012Metric_Pad1.18x1.45mm_HandSolder; Autoroute-decouple (none) -> U5
- C4: footprint (none) -> Capacitor_SMD:C_0805_2012Metric_Pad1.18x1.45mm_HandSolder; Autoroute-decouple (none) -> U2
- C5: footprint (none) -> Capacitor_SMD:C_0805_2012Metric_Pad1.18x1.45mm_HandSolder; Autoroute-decouple (none) -> U4
- U1, U2: footprint (none) -> Package_DIP:DIP-16_W7.62mm_Socket_LongPads; MPN (none) -> SN74HC283N
- U3: footprint (none) -> Package_DIP:DIP-20_W7.62mm_Socket_LongPads; MPN (none) -> SN74HC245N
- U4, U5: footprint (none) -> Package_DIP:DIP-14_W7.62mm_Socket_LongPads; MPN (none) -> SN74HC86N
Connections:
- net +5V is gone; now on net 5V: C1.2, C2.1, C3.1, C4.2, C5.2, U1.16 (VCC), U2.16 (VCC), U3.20 (VCC), U4.14 (VCC), U5.14 (VCC)
- net LABus0 is gone; now on net LBA0: U2.5 (A1)
- net LABus1 is gone; now on net LBA1: U2.3 (A2)
- net LABus2 is gone; now on net LBA2: U2.14 (A3)
- net LABus3 is gone; now on net LBA3: U2.12 (A4)
- net LABus4 is gone; now on net LBA4: U1.5 (A1)
- net LABus5 is gone; now on net LBA5: U1.3 (A2)
- net LABus6 is gone; now on net LBA6: U1.14 (A3)
- net LABus7 is gone; now on net LBA7: U1.12 (A4)
- net LBBus0 is gone; now on net LBB0: U5.2
- net LBBus1 is gone; now on net LBB1: U5.5
- net LBBus2 is gone; now on net LBB2: U5.10
- net LBBus3 is gone; now on net LBB3: U5.13
- net LBBus4 is gone; now on net LBB4: U4.2
- net LBBus5 is gone; now on net LBB5: U4.5
- net LBBus6 is gone; now on net LBB6: U4.10
- net LBBus7 is gone; now on net LBB7: U4.13
- net 5V: now also U3.1 (A->B)
- net SUM0: now also D8.2 (A); no longer D1.2 (A)
- net SUM1: now also D7.2 (A); no longer D2.2 (A)
- net SUM2: now also D6.2 (A); no longer D3.2 (A)
- net SUM3: now also D5.2 (A); no longer D4.2 (A)
- net SUM4: now also D4.2 (A); no longer D5.2 (A)
- net SUM5: now also D3.2 (A); no longer D6.2 (A)
- net SUM6: now also D2.2 (A); no longer D7.2 (A)
- net SUM7: now also D1.2 (A); no longer D8.2 (A)
- net ~{ADDO}: now also U3.19 (CE)
