File: ProgramROM/ProgramROM.kicad_pcb (KiCad board)
At the start: 2 copper layers, 85 x 99.5 mm, 41 parts, among them J2 Arduino, SW1 SW_DIP_x05, U1 AT28C64, U2 74HC541, U3 74HC595, U4 74HC245, U5 74HC157, U6 74HC04

Commit message: [ProgramRom] - added option for future Library bank within the EEProm as described in LibraryBank.md
Parts:
- added J1: LibSel, Connector_PinHeader_2.54mm:PinHeader_1x04_P2.54mm_Vertical, F.Cu at (37.1, 107.3)
- added R16: 10K, Resistor_SMD:R_0805_2012Metric_Pad1.20x1.40mm_HandSolder, F.Cu at (41.3, 104.2)
- SW1: value SW_DIP_x05 -> Program Sel (5 for Lib)
- moved R13 55.3 mm to (47.6, 111.6)
Connections:
- R13 pad 2: EE_A12 -> DIP
- SW1 pad 6: EE_A12 -> DIP
Routing:
- net EE_A12: track 92.2 -> 60.6 mm, vias 2 -> 1
- net DIP: track 0.00 -> 17.9 mm, vias 0 -> 1
- net 5V: track 280.9 -> 290.0 mm, vias 8 -> 9
- net LBA8: track 0.00 -> 6.46 mm
- net GND: track 65.4 -> 67.5 mm, vias 13 -> 14
Other:
- board text added: "Ben Eater 8-Bit Computer Program Rom v1.0 D. Q. McDonald July 2026"
- board text added: "DIP"
- board text added: "Lib"
- board text added: "LibSel (Fit Jumper)"
- board text removed: "Ben Eater 8-Bit Computer Program Rom v.0 D. Q. McDonald July 2026"
